Commit message: built ros2 package for arm_desc

File: arm_desc/urdf/robot.urdf.xacro (robot description, xacro)
@@ -1,9 +1,9 @@
 <?xml version="1.0"?>
-<robot name="robotic_arm">
+<robot name="robotic_arm" xmlns:xacro="http://www.ros.org/wiki/xacro">
 <link name="base_link">
 <visual>
 <origin xyz="0.0024960130633573558712 0.12804634114627058694 -0.01108280622936548554" rpy="0 -0 0" />
 <geometry>
-<mesh filename="package://meshes/base_link.stl"/>
+<mesh filename="package://arm_desc/meshes/base_link.stl"/>
 </geometry>
 <material name="base_link_material">
@@ -14,5 +14,5 @@
 <origin xyz="0.0024960130633573558712 0.12804634114627058694 -0.01108280622936548554" rpy="0 -0 0" />
 <geometry>
-<mesh filename="package://meshes/base_link.stl"/>
+<mesh filename="package://arm_desc/meshes/base_link.stl"/>
 </geometry>
 </collision>
@@ -27,5 +27,5 @@
 <origin xyz="0.058066221705191579938 -0.0010000035544516496996 0.035111317800536695488" rpy="-1.570796326794896558 -1.570796326794896558 0" />
 <geometry>
-<mesh filename="package://meshes/link_1.stl"/>
+<mesh filename="package://arm_desc/meshes/link_1.stl"/>
 </geometry>
 <material name="link_1_material">
@@ -36,5 +36,5 @@
 <origin xyz="0.058066221705191579938 -0.0010000035544516496996 0.035111317800536695488" rpy="-1.570796326794896558 -1.570796326794896558 0" />
 <geometry>
-<mesh filename="package://meshes/link_1.stl"/>
+<mesh filename="package://arm_desc/meshes/link_1.stl"/>
 </geometry>
 </collision>
@@ -49,5 +49,5 @@
 <origin xyz="0.058066756826188309359 0.00099999999999915933045 -0.043111317800536799738" rpy="1.570796326794896558 1.570796326794896558 0" />
 <geometry>
-<mesh filename="package://meshes/link_2.stl"/>
+<mesh filename="package://arm_desc/meshes/link_2.stl"/>
 </geometry>
 <material name="link_2_material">
@@ -58,5 +58,5 @@
 <origin xyz="0.058066756826188309359 0.00099999999999915933045 -0.043111317800536799738" rpy="1.570796326794896558 1.570796326794896558 0" />
 <geometry>
-<mesh filename="package://meshes/link_2.stl"/>
+<mesh filename="package://arm_desc/meshes/link_2.stl"/>
 </geometry>
 </collision>
@@ -71,5 +71,5 @@
 <origin xyz="-0.3889332431738120599 -0.0010000000000015309143 0.042111321354989406096" rpy="-1.570796326794896558 -1.570796326794896558 0" />
 <geometry>
-<mesh filename="package://meshes/link_3.stl"/>
+<mesh filename="package://arm_desc/meshes/link_3.stl"/>
 </geometry>
 <material name="link_3_material">
@@ -80,5 +80,5 @@
 <origin xyz="-0.3889332431738120599 -0.0010000000000015309143 0.042111321354989406096" rpy="-1.570796326794896558 -1.570796326794896558 0" />
 <geometry>
-<mesh filename="package://meshes/link_3.stl"/>
+<mesh filename="package://arm_desc/meshes/link_3.stl"/>
 </geometry>
 </collision>
@@ -93,5 +93,5 @@
 <origin xyz="-0.38893324317381300359 0.0010000000000021103119 -0.043161592520954500385" rpy="1.570796326794896558 1.570796326794896558 0" />
 <geometry>
-<mesh filename="package://meshes/link_4.stl"/>
+<mesh filename="package://arm_desc/meshes/link_4.stl"/>
 </geometry>
 <material name="link_4_material">
@@ -102,5 +102,5 @@
 <origin xyz="-0.38893324317381300359 0.0010000000000021103119 -0.043161592520954500385" rpy="1.570796326794896558 1.570796326794896558 0" />
 <geometry>
-<mesh filename="package://meshes/link_4.stl"/>
+<mesh filename="package://arm_desc/meshes/link_4.stl"/>
 </geometry>
 </collision>
@@ -115,5 +115,5 @@
 <origin xyz="0.085161592520954398911 0.0010125586032828232108 -0.42993324317381198529" rpy="1.570796326794896558 1.3040595762004301237e-18 6.4830711884908311151e-22" />
 <geometry>
-<mesh filename="package://meshes/link_5.stl"/>
+<mesh filename="package://arm_desc/meshes/link_5.stl"/>
 </geometry>
 <material name="link_5_material">
@@ -124,5 +124,5 @@
 <origin xyz="0.085161592520954398911 0.0010125586032828232108 -0.42993324317381198529" rpy="1.570796326794896558 1.3040595762004301237e-18 6.4830711884908311151e-22" />
 <geometry>
-<mesh filename="package://meshes/link_5.stl"/>
+<mesh filename="package://arm_desc/meshes/link_5.stl"/>
 </geometry>
 </collision>

Commit message: fix a bunch of stuff

File: arm_desc/urdf/robot.urdf.xacro (robot description, xacro)
@@ -138,5 +138,5 @@
 <child link="link_5" />
 <axis xyz="0 0 1"/>
-<limit effort="1" velocity="20" lower="-1.57" upper="1.57/>
+<limit effort="1" velocity="20" lower="-1.57" upper="1.57"/>
 <joint_properties friction="0.0"/>
 </joint>
@@ -146,5 +146,5 @@
 <child link="link_4" />
 <axis xyz="0 0 1"/>
-<limit effort="1" velocity="20" lower="-1.57" upper="1.57/>
+<limit effort="1" velocity="20" lower="-1.57" upper="1.57"/>
 <joint_properties friction="0.0"/>
 </joint>
@@ -154,5 +154,5 @@
 <child link="link_3" />
 <axis xyz="0 0 1"/>
-<limit effort="1" velocity="20" lower="-1.57" upper="1.57/>
+<limit effort="1" velocity="20" lower="-1.57" upper="1.57"/>
 <joint_properties friction="0.0"/>
 </joint>
@@ -162,5 +162,5 @@
 <child link="link_2" />
 <axis xyz="0 0 1"/>
-<limit effort="1" velocity="20" lower="-1.57" upper="1.57/>
+<limit effort="1" velocity="20" lower="-1.57" upper="1.57"/>
 <joint_properties friction="0.0"/>
 </joint>
@@ -170,5 +170,5 @@
 <child link="link_1" />
 <axis xyz="0 0 1"/>
-<limit effort="1" velocity="20" lower="-1.57" upper="1.57/>
+<limit effort="1" velocity="20" lower="-1.57" upper="1.57"/>
 <joint_properties friction="0.0"/>
 </joint>
